File: H7PI_Exp_Games_tft/H7PI_Exp_Games.sch (KiCad schematic (older format))
At the start: 53 parts, among them J1 Header_1x2, K1 KAN0741-0601M1, Q1 CJ2102, U1 MT9700, U10 H7PI_Exp, U11 KLJ-5018, U2 AHT10, U3 BH1730FVC-TR, U4 HP203B, U5 ME6215C33M5G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

Commit message: add tft branch Signed-off-by: fuhua-chen <fuhua-chen@outlook.com>
Parts:
- removed C10, C14: 10uF, C_1206_3216Metric, symbol capacitor:CL31B106KBHNNNE
- removed C16, C19, C21: 1uF, C_0603_1608Metric, symbol capacitor:0603B105K500NT
- removed C18, C20: 100nF, C_0402_1005Metric, symbol capacitor:0402B104K500NT
- removed D1: 1N5819WS, D_SOD-323, symbol diode:1N5819WS
- removed L1: MPH201214S100MT, L_0805_2012Metric, symbol inductor:MPH201214S100MT
- removed R10, R18: 470k, R_0402_1005Metric, symbol resistor:0402WGF470KTCE
- removed R11: 33k, R_0402_1005Metric, symbol resistor:0402WGF3302TCE
- removed R8: 10k, R_0402_1005Metric, symbol resistor:0402WGF1002TCE
- removed R9: 510k, R_0402_1005Metric, symbol resistor:0402WGF5103TCE
- removed U1: MT9700, SOT-23-5, symbol switch:MT9700
- removed U7: MT3608, SOT-23-6, symbol pmic:MT3608
- removed U8: OLED_WhiteFont_1.3Inch_128x64Pixels_35.8x17.1mm, OLED_1.3Inch_128x64Pixels_35.8x17.1x1.43mm, symbol display:OLED_WhiteFont_1.3Inch_128x64Pixels_35.8x17.1mm
- added C10: 1uF, C_0603_1608Metric, symbol capacitor:0603B105K500NT
- added C14, C16: 100nF, C_0402_1005Metric, symbol capacitor:0402B104K500NT
- added Q2: CJ2102, SOT-323_SC-70, symbol mosfet:CJ2102
- added R10: 10, R_0402_1005Metric, symbol resistor:0402WGF100JTCE
- added R8: 33k, R_0402_1005Metric, symbol resistor:0402WGF3302TCE
- added R9: 470k, R_0402_1005Metric, symbol resistor:0402WGF470KTCE
- added U1: ME6215C33M5G, SOT-23-5, symbol pmic:ME6215C33M5G
- added U7: TFT_ZJY114IPS_1.14Inch_135x240Pixels_17.6x31.0x1.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, TFT_ZJY114IPS_1.14Inch_135x240Pixels_17.6x31.0x1.6mm, symbol display:TFT_ZJY114IPS_1.14Inch_135x240Pixels_17.6x31.0x1.6mm
Connections:
- net labels added: LEDK, TFT_3V3, TFT_BL, TFT_EN
- net labels removed: 9V, IREF, OLED_EN
- wire segments 292 -> 255
- no-connect marks 38 -> 35

Commit message: v0.2 update expansion board symbol and footprint
Signed-off-by: fuhua-chen <fuhua-chen@outlook.com>
Connections:
- no-connect marks 35 -> 37
Changed lines of the file:
@@
 Text Label 10950 2300 2    50   ~ 0
 TFT_BL
+NoConn ~ 8250 2100
+NoConn ~ 9100 2100
 $EndSCHEMATC
